Commit message: Add arduino hardware interface

File: src/robot/description/gazebo_control.xacro (robot description, xacro)
@@ -2,5 +2,5 @@
 <robot xmlns:xacro="http://www.ros.org/wiki/xacro">
     <gazebo>
-        <plugin name="diff_drive" filename="libgazebo_ros_diff_drive.so">
+        <plugin name="gazebo_ros_diff_drive" filename="libgazebo_ros_diff_drive.so">
             <!-- Wheel information -->
             <left_joint>left_wheel_joint</left_joint>  <!-- Name of the left wheel joint -->

File: src/robot/description/ros2_control.xacro (robot description, xacro)
@@ -1,8 +1,14 @@
 <?xml version="1.0"?>
 <robot xmlns:xacro="http://www.ros.org/wiki/xacro">
-    <!-- Define hardware interface for the controller manager -->
-    <ros2_control name="GazeboSystem" type="system">
+    <ros2_control name="ros_diff_drive" type="system">
         <hardware>
-            <plugin>gazebo_ros2_control/GazeboSystem</plugin>
+            <plugin>diffdrive_arduino/DiffDriveArduino</plugin>
+            <param name="left_wheel_name">left_wheel_joint</param>
+            <param name="right_wheel_name">right_wheel_joint</param>
+            <param name="loop_rate">30</param>
+            <param name="device">/dev/ttyUSB0</param>
+            <param name="baud_rate">57600</param>
+            <param name="timeout">1000</param>
+            <param name="enc_counts_per_rev">2000</param>
         </hardware>
         <joint name="left_wheel_joint">
@@ -25,4 +31,28 @@
         </joint>
     </ros2_control>
+    <!-- Define hardware interface for the controller manager
+    <ros2_control name="GazeboSystem" type="system">
+        <hardware>
+            <plugin>gazebo_ros2_control/GazeboSystem</plugin>
+        </hardware>
+        <joint name="left_wheel_joint">
+            <command_interface name="velocity">
+                Set up the minimum and maximum velocity values
+                <param name="min">-10</param>
+                <param name="max">10</param>
+            </command_interface>
+            Specify the state interfaces providing the velocity and position of the joint
+            <state_interface name="velocity"/>
+            <state_interface name="position"/>
+        </joint>
+        <joint name="right_wheel_joint">
+            <command_interface name="velocity">
+                <param name="min">-10</param>
+                <param name="max">10</param>
+            </command_interface>
+            <state_interface name="velocity"/>
+            <state_interface name="position"/>
+        </joint>
+    </ros2_control> -->
     <!-- Tells Gazebo o use ros2 control.
     Note that his plugin runs its own controller manager -->
