Commit message: Identify motor controller device file dynamically

File: src/robot/description/ros2_control.xacro (robot description, xacro)
@@ -1,4 +1,5 @@
 <?xml version="1.0"?>
 <robot xmlns:xacro="http://www.ros.org/wiki/xacro">
+    <xacro:property name="device" value="$(arg device)"/>
     <xacro:unless value="$(arg sim_mode)">
         <ros2_control name="RosDiffDrive" type="system">
@@ -8,5 +9,5 @@
                 <param name="right_wheel_name">right_wheel_joint</param>
                 <param name="loop_rate">30</param>
-                <param name="device">/dev/ttyUSB0</param>
+                <param name="device">${device}</param>
                 <param name="baud_rate">57600</param>
                 <param name="timeout">1000</param>
